Commit message: Specified correct path

File: urdf/my_robot.xacro (robot description, xacro)
@@ -180,5 +180,5 @@
       <origin xyz="0 0 0" rpy=" 0 0 0"/>
       <geometry>
-        <mesh filename="package://my_robot/meshes/hokuyo.dae"/>
+        <mesh filename="package://udacity_bot/meshes/hokuyo.dae"/>
       </geometry>
     </visual>
